Commit message: imporve visualization (fix scale of forces, add motors to urdf, add Fl, Fd, Fs publishers), add new tests fix axis a little bit

File: urdf/vtol.urdf.xacro (robot description, xacro)
@@ -1,8 +1,17 @@
 <?xml version="1.0"?>
 <robot name="vtol" xmlns:xacro="http://www.ros.org/wiki/xacro">
-  <xacro:property name="BASE_LENGTH"      value="0.890" />
-  <xacro:property name="BASE_WIDTH"       value="0.596" />
-  <xacro:property name="BASE_HEIGHT"      value="0.1" />
-  <xacro:property name="BASE_MASS"        value="7" />
+  <xacro:property name="PROP_LOCATION_X"    value="0.445" />
+  <xacro:property name="PROP_LOCATION_Y"    value="0.422" />
+  <xacro:property name="PROP_LOCATION_Z"    value="0.01" />
+  <xacro:property name="ICE_RADIUS"         value="0.1" />
+  <xacro:property name="ICE_WIDTH"          value="0.05" />
+  <xacro:property name="MOTOR_RADIUS"       value="0.1" />
+  <xacro:property name="MOTOR_WIDTH"        value="0.01" />
+  <material name="grey">
+    <color rgba="0.5 0.5 0.5 1.0"/>
+  </material>
+  <material name="light_black">
+    <color rgba="0.4 0.4 0.4 1.0"/>
+  </material>
   <link name="base_footprint"/>
   <link name="base_link">
@@ -10,5 +19,5 @@
       <origin xyz="0 0 0" />
       <geometry>
-        <box size="${BASE_LENGTH} ${BASE_WIDTH} ${BASE_HEIGHT}"/>
+        <box size="${PROP_LOCATION_X * 2} ${PROP_LOCATION_Y * 2} ${PROP_LOCATION_Z * 2}"/>
       </geometry>
       <material name="grey"/>
@@ -17,5 +26,5 @@
       <origin xyz="0 0 0" rpy="0 0 0"/>
       <geometry>
-        <box size="${BASE_LENGTH} ${BASE_WIDTH} ${BASE_HEIGHT}"/>
+        <box size="${PROP_LOCATION_X * 2} ${PROP_LOCATION_Y * 2} ${PROP_LOCATION_Z * 2}"/>
       </geometry>
     </collision>
@@ -26,8 +35,108 @@
     <origin xyz="0 0 0" rpy="0 0 0"/>
   </joint>
-  <gazebo reference="base_link">
-    <material>Gazebo/Grey</material>
-    <turnGravityOff>false</turnGravityOff>
-    <selfCollide>false</selfCollide>
-  </gazebo>
+  <link name="ICE">
+    <visual>
+      <origin xyz="0 0 0" rpy="0 1.57 0"/>
+      <geometry>
+        <cylinder radius="${ICE_RADIUS}" length="${ICE_WIDTH}" />
+      </geometry>
+      <material name="light_black"/>
+    </visual>
+    <collision>
+      <origin xyz="0 0 0"/>
+      <geometry>
+        <cylinder radius="${ICE_RADIUS}" length="${ICE_WIDTH}" />
+      </geometry>
+    </collision>
+  </link>
+  <joint name="ice_connect" type="fixed">
+    <parent link="base_link"/>
+    <child link="ICE"/>
+    <origin xyz="${PROP_LOCATION_X} 0.0 0.0" rpy="0 0 0"/>
+    <axis xyz="0 0 1"/>
+  </joint>
+  <link name="motor0">
+    <visual>
+      <origin xyz="0 0 0" rpy="0 0 0"/>
+      <geometry>
+        <cylinder radius="${MOTOR_RADIUS}" length="${MOTOR_WIDTH}" />
+      </geometry>
+      <material name="light_black"/>
+    </visual>
+    <collision>
+      <origin xyz="0 0 0"/>
+      <geometry>
+        <cylinder radius="${MOTOR_RADIUS}" length="${MOTOR_WIDTH}" />
+      </geometry>
+    </collision>
+  </link>
+  <joint name="motor0_connect" type="fixed">
+    <parent link="base_link"/>
+    <child link="motor0"/>
+    <origin xyz="${PROP_LOCATION_X * 0.707} ${PROP_LOCATION_Y * 0.707} ${PROP_LOCATION_Z}" rpy="0 0 0"/>
+    <axis xyz="0 0 1"/>
+  </joint>
+  <link name="motor1">
+    <visual>
+      <origin xyz="0 0 0" rpy="0 0 0"/>
+      <geometry>
+        <cylinder radius="${MOTOR_RADIUS}" length="${MOTOR_WIDTH}" />
+      </geometry>
+      <material name="light_black"/>
+    </visual>
+    <collision>
+      <origin xyz="0 0 0"/>
+      <geometry>
+        <cylinder radius="${MOTOR_RADIUS}" length="${MOTOR_WIDTH}" />
+      </geometry>
+    </collision>
+  </link>
+  <joint name="motor1_connect" type="fixed">
+    <parent link="base_link"/>
+    <child link="motor1"/>
+    <origin xyz="${-PROP_LOCATION_X * 0.707} ${-PROP_LOCATION_Y * 0.707} ${PROP_LOCATION_Z}" rpy="0 0 0"/>
+    <axis xyz="0 0 1"/>
+  </joint>
+  <link name="motor2">
+    <visual>
+      <origin xyz="0 0 0" rpy="0 0 0"/>
+      <geometry>
+        <cylinder radius="${MOTOR_RADIUS}" length="${MOTOR_WIDTH}" />
+      </geometry>
+      <material name="light_black"/>
+    </visual>
+    <collision>
+      <origin xyz="0 0 0"/>
+      <geometry>
+        <cylinder radius="${MOTOR_RADIUS}" length="${MOTOR_WIDTH}" />
+      </geometry>
+    </collision>
+  </link>
+  <joint name="motor2_connect" type="fixed">
+    <parent link="base_link"/>
+    <child link="motor2"/>
+    <origin xyz="${PROP_LOCATION_X * 0.707} ${-PROP_LOCATION_Y * 0.707} ${PROP_LOCATION_Z}" rpy="0 0 0"/>
+    <axis xyz="0 0 1"/>
+  </joint>
+  <link name="motor3">
+    <visual>
+      <origin xyz="0 0 0" rpy="0 0 0"/>
+      <geometry>
+        <cylinder radius="${MOTOR_RADIUS}" length="${MOTOR_WIDTH}" />
+      </geometry>
+      <material name="light_black"/>
+    </visual>
+    <collision>
+      <origin xyz="0 0 0"/>
+      <geometry>
+        <cylinder radius="${MOTOR_RADIUS}" length="${MOTOR_WIDTH}" />
+      </geometry>
+    </collision>
+  </link>
+  <joint name="motor3_connect" type="fixed">
+    <parent link="base_link"/>
+    <child link="motor3"/>
+    <origin xyz="${-PROP_LOCATION_X * 0.707} ${PROP_LOCATION_Y * 0.707} ${PROP_LOCATION_Z}" rpy="0 0 0"/>
+    <axis xyz="0 0 1"/>
+  </joint>
 </robot>

Commit message: fix calibration initial orientations and visualization in rviz

File: urdf/vtol.urdf.xacro (robot description, xacro)
@@ -17,7 +17,7 @@
   <link name="base_link">
     <visual>
-      <origin xyz="0 0 0" />
+      <origin xyz="0 0 0" rpy="3.14 0 3.14"/>
       <geometry>
-        <box size="${PROP_LOCATION_X * 2} ${PROP_LOCATION_Y * 2} ${PROP_LOCATION_Z * 2}"/>
+        <mesh filename="package://innopolis_vtol_dynamics/meshes/vtol.dae" scale="0.00333 0.00333 0.00333"/>
       </geometry>
       <material name="grey"/>
@@ -36,11 +36,4 @@
   </joint>
   <link name="ICE">
-    <visual>
-      <origin xyz="0 0 0" rpy="0 1.57 0"/>
-      <geometry>
-        <cylinder radius="${ICE_RADIUS}" length="${ICE_WIDTH}" />
-      </geometry>
-      <material name="light_black"/>
-    </visual>
     <collision>
       <origin xyz="0 0 0"/>
@@ -57,11 +50,4 @@
   </joint>
   <link name="motor0">
-    <visual>
-      <origin xyz="0 0 0" rpy="0 0 0"/>
-      <geometry>
-        <cylinder radius="${MOTOR_RADIUS}" length="${MOTOR_WIDTH}" />
-      </geometry>
-      <material name="light_black"/>
-    </visual>
     <collision>
       <origin xyz="0 0 0"/>
@@ -78,11 +64,4 @@
   </joint>
   <link name="motor1">
-    <visual>
-      <origin xyz="0 0 0" rpy="0 0 0"/>
-      <geometry>
-        <cylinder radius="${MOTOR_RADIUS}" length="${MOTOR_WIDTH}" />
-      </geometry>
-      <material name="light_black"/>
-    </visual>
     <collision>
       <origin xyz="0 0 0"/>
@@ -99,11 +78,4 @@
   </joint>
   <link name="motor2">
-    <visual>
-      <origin xyz="0 0 0" rpy="0 0 0"/>
-      <geometry>
-        <cylinder radius="${MOTOR_RADIUS}" length="${MOTOR_WIDTH}" />
-      </geometry>
-      <material name="light_black"/>
-    </visual>
     <collision>
       <origin xyz="0 0 0"/>
@@ -120,11 +92,4 @@
   </joint>
   <link name="motor3">
-    <visual>
-      <origin xyz="0 0 0" rpy="0 0 0"/>
-      <geometry>
-        <cylinder radius="${MOTOR_RADIUS}" length="${MOTOR_WIDTH}" />
-      </geometry>
-      <material name="light_black"/>
-    </visual>
     <collision>
       <origin xyz="0 0 0"/>

Commit message: add mesh for VTOL model and update urdf file

File: urdf/vtol.urdf.xacro (robot description, xacro)
@@ -19,5 +19,5 @@
       <origin xyz="0 0 0" rpy="3.14 0 3.14"/>
       <geometry>
-        <mesh filename="package://innopolis_vtol_dynamics/meshes/vtol.dae" scale="0.00333 0.00333 0.00333"/>
+        <mesh filename="package://innopolis_vtol_dynamics/meshes/vtol.stl" scale="0.00333 0.00333 0.00333"/>
       </geometry>
       <material name="grey"/>
